File: design/kicad/display_MSP2807.kicad_sch (KiCad schematic)
At the start: 2 parts

Commit message: Fix net format name and update junctions in MIDI controller schematic
- Set net format name to "KiCad" in the project file.
- Added multiple junctions at specified coordinates in the schematic.
- Adjusted existing junction positions and UUIDs for consistency.
- Updated wire connections to reflect new junction placements.
- Corrected component references and properties for various components.
- Added new capacitor symbols with appropriate properties and references.
Parts:
- added C9: 10uF_0805_16V_lowESR, Capacitor_SMD:C_0805_2012Metric, symbol PCM_4ms_Capacitor:10uF_0805_16V_lowESR
- renumbered C2 to C8, D1 to D40
Connections:
- net +5V: now also C9.1
- net GND: now also C9.2
Changed lines of the file:
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@@
+	)
+	(junction
+		(at 170.18 62.23)
+		(diameter 0)
+		(color 0 0 0 0)
+	)
+	(junction
+		(at 170.18 74.93)
+		(diameter 0)
+		(color 0 0 0 0)
 	)
 	(junction
@@
 	(wire
 		(pts
+			(xy 170.18 62.23) (xy 170.18 66.04)
+		)
+		(stroke
+			(width 0)
+			(type default)
+		)
+	)
+	(wire
+		(pts
 			(xy 152.4 72.39) (xy 154.94 72.39)
 		)
@@
 	(wire
 		(pts
+			(xy 170.18 74.93) (xy 173.99 74.93)
+		)
+		(stroke
+			(width 0)
+			(type default)
+		)
+	)
+	(wire
+		(pts
 			(xy 152.4 90.17) (xy 157.48 90.17)
 		)
@@
 	(wire
 		(pts
+			(xy 170.18 62.23) (xy 173.99 62.23)
+		)
+		(stroke
+			(width 0)
+			(type default)
+		)
+	)
+	(wire
+		(pts
 			(xy 154.94 62.23) (xy 160.02 62.23)
 		)
@@
 		)
 	)
+	(wire
+		(pts
+			(xy 170.18 71.12) (xy 170.18 74.93)
+		)
+		(stroke
+			(width 0)
+			(type default)
+		)
+	)
 	(global_label "GND"
 		(shape input)
-		(at 170.18 74.93 0)
+		(at 173.99 74.93 0)
 		(fields_autoplaced yes)
 		(effects
@@
 		)
 		(property "Intersheetrefs" "${INTERSHEET_REFS}"
-			(at 177.0357 74.93 0)
+			(at 180.8457 74.93 0)
 			(effects
 				(font
@@
 	(hierarchical_label "+5V"
 		(shape input)
-		(at 170.18 62.23 0)
+		(at 173.99 62.23 0)
 		(effects
 			(font
@@
 			)
 			(justify left)
+		)
+	)
+	(symbol
+		(lib_id "PCM_4ms_Capacitor:10uF_0805_16V_lowESR")
+		(at 170.18 68.58 0)
+		(unit 1)
+		(exclude_from_sim no)
+		(in_bom yes)
+		(on_board yes)
+		(dnp no)
+		(fields_autoplaced yes)
+		(property "Reference" "C9"
+			(at 172.72 67.3162 0)
+			(effects
+				(font
+					(size 1.27 1.27)
+				)
+				(justify left)
+			)
+		)
+		(property "Value" "10uF_0805_16V_lowESR"
+			(at 170.18 64.77 0)
+			(effects
+				(font
+					(size 1.27 1.27)
+				)
+				(hide yes)
+			)
+		)
+		(property "Footprint" "Capacitor_SMD:C_0805_2012Metric"
+			(at 167.64 73.66 0)
+			(effects
+				(font
+					(size 1.27 1.27)
+				)
+				(justify left)
+				(hide yes)
+			)
+		)
+		(property "Datasheet" ""
+			(at 170.18 68.58 0)
+			(effects
+				(font
+					(size 1.27 1.27)
+				)
+				(hide yes)
+			)
+		)
+		(property "Description" "10uF, Min. 16V, ESR<=20mΩ@1MHz, 0805, MLCC"
+			(at 170.18 68.58 0)
+			(effects
+				(font
+					(size 1.27 1.27)
+				)
+				(hide yes)
+			)
+		)
+		(property "Specifications" "10uF, Min. 16V, ESR<=20mΩ@1MHz, 0805, MLCC"
+			(at 167.64 76.454 0)
+			(effects
+				(font
+					(size 1.27 1.27)
+				)
+				(justify left)
+				(hide yes)
+			)
+		)
+		(property "Manufacturer" "Taiyo Yuden"
+			(at 167.64 77.978 0)
+			(effects
+				(font
+					(size 1.27 1.27)
+				)
+				(justify left)
+				(hide yes)
+			)
+		)
+		(property "Part Number" "EMK212ABJ106KG-T"
+			(at 167.64 79.502 0)
+			(effects
+				(font
+					(size 1.27 1.27)
+				)
+				(justify left)
+				(hide yes)
+			)
+		)
+		(property "Display" "10u"
+			(at 172.72 69.8562 0)
+			(effects
+				(font
+					(size 1.27 1.27)
+				)
+				(justify left)
+			)
+		)
+		(property "JLCPCB ID" "C190442"
+			(at 170.18 68.58 0)
+			(effects
+				(font
+					(size 1.27 1.27)
+				)
+				(hide yes)
+			)
+		)
+		(pin "1"
+		)
+		(pin "2"
+		)
+		(instances
+			(project ""
+				(path "/9e44e663-00d0-4f33-bf1f-c4ad78deb554/b074c366-2f0b-4fcc-8b9f-7590ca8943b4"
+					(reference "C9")
+					(unit 1)
+				)
+			)
 		)
 	)
@@
 		(on_board yes)
 		(dnp no)
-		(property "Reference" "D1"
+		(property "Reference" "D40"
 			(at 121.92 68.58 0)
 			(effects
@@
 			(project "midi_controller"
 				(path "/9e44e663-00d0-4f33-bf1f-c4ad78deb554/b074c366-2f0b-4fcc-8b9f-7590ca8943b4"
-					(reference "D1")
+					(reference "D40")
 					(unit 1)
 				)
@@
 		(dnp no)
 		(fields_autoplaced yes)
-		(property "Reference" "C2"
+		(property "Reference" "C8"
 			(at 163.83 67.3099 0)
 			(effects
@@
 			(project "midi_controller"
 				(path "/9e44e663-00d0-4f33-bf1f-c4ad78deb554/b074c366-2f0b-4fcc-8b9f-7590ca8943b4"
-					(reference "C2")
+					(reference "C8")
 					(unit 1)
 				)
