File: design/kicad/_OLD/midi_controller.kicad_pcb (KiCad board)
At the start: 4 copper layers, 166 x 166 mm, 123 parts, among them J1 Conn_01x05, J10 Conn_01x24_Socket, J2 Conn_01x02_Socket, J3 Conn_01x02_Socket, J4 Conn_01x02_Socket, J5 Conn_01x02_Socket, J6 Conn_01x02_Socket, J7 Conn_01x02_Socket, J9 Conn_01x24_Socket, U1 CD74HC4067M

Commit message: Update kicad binary files
Parts:
- removed the C22 at (207.0, 176.7)
- removed the C23 at (207.1, 181.7)
- removed the C24 at (231.6, 178.3)
- removed the C25 at (112.5, 221.7)
- removed the C26 at (112.6, 216.7)
- removed the C27 at (88.5, 221.7)
- removed the C28 at (152.3, 221.8)
- removed the C29 at (152.3, 216.8)
- removed the C30 at (128.2, 221.8)
- removed the C31 at (167.6, 216.7)
- removed the C32 at (167.6, 221.7)
- removed the C33 at (191.7, 218.3)
- removed the C34 at (207.1, 216.7)
- removed the C35 at (207.1, 221.7)
- removed the C39 at (231.8, 89.2)
- added C1: 100nF, PCM_JLCPCB:C_0603, F.Cu at (206.7, 94.2)
- added C10: 100nF, PCM_JLCPCB:C_0603, F.Cu at (167.6, 181.7)
- added C11: 100nF, PCM_JLCPCB:C_0603, F.Cu at (167.5, 176.8)
- added C12: 100nF, PCM_JLCPCB:C_0603, F.Cu at (207.0, 176.7)
- added C13: 100nF, PCM_JLCPCB:C_0603, F.Cu at (207.1, 181.7)
- added C14: 100nF, PCM_JLCPCB:C_0603, F.Cu at (112.7, 221.7)
- added C15: 100nF, PCM_JLCPCB:C_0603, F.Cu at (112.7, 216.7)
- added C2: 100nF, PCM_JLCPCB:C_0603, F.Cu at (206.8, 89.2)
- added C3: 100nF, PCM_JLCPCB:C_0603, F.Cu at (231.9, 89.2)
- added C40: 100nF, PCM_JLCPCB:C_0603, B.Cu at (231.7, 218.2)
- added C41: 100nF, PCM_JLCPCB:C_0603, B.Cu at (191.9, 218.3)
- added C42: 100nF, PCM_JLCPCB:C_0603, B.Cu at (128.0, 221.8)
- added C43: 100nF, PCM_JLCPCB:C_0603, B.Cu at (88.5, 221.8)
- added C8: 100nF, PCM_JLCPCB:C_0603, F.Cu at (151.9, 181.8)
- added C9: 100nF, PCM_JLCPCB:C_0603, F.Cu at (152.3, 176.8)
- C16, C17, C19, C20, C36: value 100n -> 100nF; footprint Capacitor_SMD:C_0603_1608Metric -> PCM_JLCPCB:C_0603
- C18, C21: value 100n -> 100nF; footprint Capacitor_SMD:C_0603_1608Metric -> PCM_JLCPCB:C_0603; moved to F.Cu
- C23: renamed from C8; value 100n -> 100nF; footprint Capacitor_SMD:C_0805_2012Metric -> PCM_JLCPCB:C_0805
- C24: renamed from C6; value 10n -> 10nF; footprint Capacitor_SMD:C_0603_1608Metric -> PCM_JLCPCB:C_0603
- C25: renamed from C10; value 47u -> 47uF; footprint Capacitor_SMD:C_1206_3216Metric -> PCM_JLCPCB:C_0805
- C26: renamed from C12; value 100u -> 100uF; footprint Capacitor_SMD:C_1210_3225Metric -> PCM_JLCPCB:C_1206
- C27: renamed from C5; value 1n -> 1nF; footprint Capacitor_SMD:C_0603_1608Metric -> PCM_JLCPCB:C_0603
- C30: renamed from C2; value 10u -> 10uF; footprint Capacitor_SMD:C_0805_2012Metric -> PCM_JLCPCB:C_0805
- C31: renamed from C11; value 47u -> 47uF; footprint Capacitor_SMD:C_1206_3216Metric -> PCM_JLCPCB:C_0805
- C32: renamed from C4; value 100n -> 100nF; footprint Capacitor_SMD:C_0603_1608Metric -> PCM_JLCPCB:C_0805
- C33: renamed from C3; value 100n -> 100nF; footprint Capacitor_SMD:C_0603_1608Metric -> PCM_JLCPCB:C_0805
- C34: renamed from C7; value 1n -> 1nF; footprint Capacitor_SMD:C_0603_1608Metric -> PCM_JLCPCB:C_0603
- C35: renamed from C9; value 100n -> 100nF; footprint Capacitor_SMD:C_0805_2012Metric -> PCM_JLCPCB:C_0805
- C37, C38: value 100n -> 100nF; footprint Capacitor_SMD:C_0603_1608Metric -> PCM_JLCPCB:C_0603; moved to B.Cu
- C39: renamed from C15; value 100n -> 100nF; footprint Capacitor_SMD:C_0603_1608Metric -> PCM_JLCPCB:C_0603
- C6: renamed from C14; value 100n -> 100nF; footprint Capacitor_SMD:C_0603_1608Metric -> PCM_JLCPCB:C_0603
- C7: renamed from C13; value 100n -> 100nF; footprint Capacitor_SMD:C_0603_1608Metric -> PCM_JLCPCB:C_0603
- D25: renamed from D1; footprint Diode_SMD:D_SMA -> PCM_JLCPCB:D_SMA
- FB1, FB2, FB3, FB4: value FerriteBead -> ~; footprint Inductor_SMD:L_0805_2012Metric -> PCM_JLCPCB:FB_0805
- R1: renamed from R6; value 33 -> 33Ω; footprint Resistor_SMD:R_0603_1608Metric -> PCM_JLCPCB:R_0603
- R6: renamed from R9; value 33 -> 33Ω; footprint Resistor_SMD:R_0603_1608Metric -> PCM_JLCPCB:R_0603
- R7: renamed from R8; value 33 -> 33Ω; footprint Resistor_SMD:R_0603_1608Metric -> PCM_JLCPCB:R_0603
- R8: renamed from R5; value 33 -> 33Ω; footprint Resistor_SMD:R_0603_1608Metric -> PCM_JLCPCB:R_0603
- moved C38 117.9 mm to (127.9, 181.8)
- moved C37 90.6 mm to (191.6, 178.6), turned to 90 degrees
- moved C18 52.8 mm to (167.5, 216.7)
- moved C20 52.7 mm to (207.0, 216.7)
- moved C21 45.8 mm to (206.9, 221.7), turned to -90 degrees
- moved C19 45.0 mm to (167.6, 221.7)
- moved C17 40.0 mm to (152.2, 216.8)
- moved C16 40.0 mm to (152.2, 221.8)
- moved C36 40.0 mm to (231.6, 178.3)
- moved C32 0.81 mm to (130.8, 118.1)
- moved FB3 0.69 mm to (130.8, 120.1)
- moved C34 0.60 mm to (128.0, 122.7)
- moved C35 0.60 mm to (129.9, 122.9)
- moved C33 0.49 mm to (133.7, 119.0)
- moved C31 0.40 mm to (138.2, 119.0)
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- renumbered C1 to C22, C40 to C28, C41 to C29, C43 to C4, C42 to C5, D27 to D1, D6 to D10, D7 to D11, D9 to D12, D10 to D13, D13 to D14, D12 to D15, D15 to D16, D16 to D17, D19 to D18, D18 to D19, D29 to D2, D22 to D20, D24 to D22, D25 to D23, D2 to D24, D35 to D26, D34 to D27, D30 to D28, D31 to D29, D37 to D3, D33 to D30, D32 to D31, D14 to D32, D11 to D33, D8 to D34, D5 to D35, D26 to D36, D23 to D37, D20 to D38, D17 to D39, D36 to D4, D39 to D5, D38 to D6, D28 to D7, D4 to D8, D3 to D9, ENC_MECH9 to ENC_MECH1, ENC_MECH1 to ENC_MECH2, ENC_MECH2 to ENC_MECH3, ENC_MECH3 to ENC_MECH4, ENC_MECH4 to ENC_MECH5, ENC_MECH5 to ENC_MECH6, ENC_MECH6 to ENC_MECH7, ENC_MECH7 to ENC_MECH8, ENC_MECH8 to ENC_MECH9, J9 to J1, J3 to J2, J2 to J3, J10 to J4, J4 to J5, J1 to J6, J5 to J7, J6 to J8, J7 to J9, R4 to R2, R2 to R3, R3 to R4, R7 to R5, R1 to R9, SW3 to SW2, SW5 to SW3, SW2 to SW4, SW4 to SW5
Connections:
- C16 pad 2: /MIDI_Encoder_Matrix_2x4_with_push_buttons/1x2.QUAD_A -> /MIDI_Encoder_Matrix_2x4_with_push_buttons/2x2.QUAD_A
- C17 pad 2: /MIDI_Encoder_Matrix_2x4_with_push_buttons/1x2.QUAD_B -> /MIDI_Encoder_Matrix_2x4_with_push_buttons/2x2.QUAD_B
- C18 pad 2: /MIDI_Encoder_Matrix_2x4_with_push_buttons/1x2_SW_A -> /MIDI_Encoder_Matrix_2x4_with_push_buttons/2x3.QUAD_A
- C19 pad 2: /MIDI_Encoder_Matrix_2x4_with_push_buttons/1x3.QUAD_A -> /MIDI_Encoder_Matrix_2x4_with_push_buttons/2x3.QUAD_B
- C20 pad 2: /MIDI_Encoder_Matrix_2x4_with_push_buttons/1x3.QUAD_B -> /MIDI_Encoder_Matrix_2x4_with_push_buttons/2x4.QUAD_A
- C21 pad 2: /MIDI_Encoder_Matrix_2x4_with_push_buttons/1x3_SW_A -> /MIDI_Encoder_Matrix_2x4_with_push_buttons/2x4.QUAD_B
- C36 pad 2: /MIDI_Encoder_Matrix_2x4_with_push_buttons/2x4_SW_A -> /MIDI_Encoder_Matrix_2x4_with_push_buttons/1x4_SW_A
- C37 pad 2: /NAV.QUAD_A -> /MIDI_Encoder_Matrix_2x4_with_push_buttons/1x3_SW_A
- C38 pad 2: /NAV.QUAD_B -> /MIDI_Encoder_Matrix_2x4_with_push_buttons/1x2_SW_A
- D25 pad 2: Net-(D1-A) -> Net-(D25-Pad2)
- FB2 pad 1: Net-(D1-A) -> +5V
- FB2 pad 2: +5V -> Net-(D25-Pad2)
Routing:
- net Net-(D25-Pad2): track 0.00 -> 2.24 mm
- net Net-(D1-A): track 2.24 -> 0.00 mm
Other:
- board text added: "SD Card"
- board text added: "Teensy 4.1"
- board text added: "USB"
